Commit message: fixes

File: lizi_urdf/robots/lizi.xacro (robot description, xacro)
@@ -2,5 +2,5 @@
 <robot xmlns:xacro="http://www.ros.org/wiki/lizi" name="lizi_urdf">
   <link
-    name="lizi_$(arg lizi_id)/base_link">
+    name="lizi_$(arg lizi_id)_base_link">
     <inertial>
       <origin
@@ -42,5 +42,5 @@
   </link>
   <link
-    name="lizi_$(arg lizi_id)/FL_Wheel_Link">
+    name="lizi_$(arg lizi_id)_FL_Wheel_link">
     <inertial>
       <origin
@@ -82,5 +82,5 @@
   </link>
   <joint
-    name="lizi_$(arg lizi_id)/FL_Wheel_Joint"
+    name="lizi_$(arg lizi_id)_FL_Wheel_Joint"
     type="continuous">
     <origin
@@ -88,12 +88,12 @@
       rpy="0 0 -1.3371E-16" />
     <parent
-      link="lizi_$(arg lizi_id)/base_link" />
-    <child
-      link="lizi_$(arg lizi_id)/FL_Wheel_Link" />
+      link="lizi_$(arg lizi_id)_base_link" />
+    <child
+      link="lizi_$(arg lizi_id)_FL_Wheel_link" />
     <axis
       xyz="0 -1 0" />
   </joint>
   <link
-    name="lizi_$(arg lizi_id)/RL_Wheel_Link">
+    name="lizi_$(arg lizi_id)_RL_Wheel_link">
     <inertial>
       <origin
@@ -135,5 +135,5 @@
   </link>
   <joint
-    name="lizi_$(arg lizi_id)/RL_Wheel_Joint"
+    name="lizi_$(arg lizi_id)_RL_Wheel_Joint"
     type="continuous">
     <origin
@@ -141,7 +141,7 @@
       rpy="0 0 -6.6853E-16" />
     <parent
-      link="lizi_$(arg lizi_id)/base_link" />
-    <child
-      link="lizi_$(arg lizi_id)/RL_Wheel_Link" />
+      link="lizi_$(arg lizi_id)_base_link" />
+    <child
+      link="lizi_$(arg lizi_id)_RL_Wheel_link" />
     <axis
       xyz="0 -1 0" />
@@ -151,5 +151,5 @@
   </joint>
   <link
-    name="lizi_$(arg lizi_id)/RR_Wheel_Link">
+    name="lizi_$(arg lizi_id)_RR_Wheel_link">
     <inertial>
       <origin
@@ -191,5 +191,5 @@
   </link>
   <joint
-    name="lizi_$(arg lizi_id)/RR_Wheel_Joint"
+    name="lizi_$(arg lizi_id)_RR_Wheel_Joint"
     type="continuous">
     <origin
@@ -197,12 +197,12 @@
       rpy="-1.2938E-16 -1.2938E-15 -6.6853E-16" />
     <parent
-      link="lizi_$(arg lizi_id)/base_link" />
-    <child
-      link="lizi_$(arg lizi_id)/RR_Wheel_Link" />
+      link="lizi_$(arg lizi_id)_base_link" />
+    <child
+      link="lizi_$(arg lizi_id)_RR_Wheel_link" />
     <axis
       xyz="0 1 0" />
   </joint>
   <link
-    name="lizi_$(arg lizi_id)/FR_Wheel_Link">
+    name="lizi_$(arg lizi_id)_FR_Wheel_link">
     <inertial>
       <origin
@@ -244,5 +244,5 @@
   </link>
   <joint
-    name="lizi_$(arg lizi_id)/FR_Wheel_Joint"
+    name="lizi_$(arg lizi_id)_FR_Wheel_Joint"
     type="continuous">
     <origin
@@ -250,12 +250,12 @@
       rpy="4.4216E-16 -0.0061583 -2.6824E-16" />
     <parent
-      link="lizi_$(arg lizi_id)/base_link" />
-    <child
-      link="lizi_$(arg lizi_id)/FR_Wheel_Link" />
+      link="lizi_$(arg lizi_id)_base_link" />
+    <child
+      link="lizi_$(arg lizi_id)_FR_Wheel_link" />
     <axis
       xyz="0 1 0" />
   </joint>
   <link
-    name="lizi_$(arg lizi_id)/Asus_Pan_Link">
+    name="lizi_$(arg lizi_id)_Asus_Pan_link">
     <inertial>
       <origin
@@ -297,5 +297,5 @@
   </link>
   <joint
-    name="lizi_$(arg lizi_id)/Asus_Pan_Joint"
+    name="lizi_$(arg lizi_id)_Asus_Pan_Joint"
     type="revolute">
     <origin
@@ -303,7 +303,7 @@
       rpy="2.1253E-16 8.5011E-16 0" />
     <parent
-      link="lizi_$(arg lizi_id)/base_link" />
-    <child
-      link="lizi_$(arg lizi_id)/Asus_Pan_Link" />
+      link="lizi_$(arg lizi_id)_base_link" />
+    <child
+      link="lizi_$(arg lizi_id)_Asus_Pan_link" />
     <axis
       xyz="0 0 -1" />
@@ -313,5 +313,5 @@
   </joint>
   <link
-    name="lizi_$(arg lizi_id)/Asus_Camera_Link">
+    name="lizi_$(arg lizi_id)_Asus_Camera_link">
     <inertial>
       <origin
@@ -353,5 +353,5 @@
   </link>
   <joint
-    name="lizi_$(arg lizi_id)/Asus_Tilt_Joint"
+    name="lizi_$(arg lizi_id)_Asus_Tilt_Joint"
     type="revolute">
     <origin
@@ -359,7 +359,7 @@
       rpy="1.5708 -8.5011E-16 1.8067E-31" />
     <parent
-      link="lizi_$(arg lizi_id)/Asus_Pan_Link" />
-    <child
-      link="lizi_$(arg lizi_id)/Asus_Camera_Link" />
+      link="lizi_$(arg lizi_id)_Asus_Pan_link" />
+    <child
+      link="lizi_$(arg lizi_id)_Asus_Camera_link" />
     <axis
       xyz="-0.027278 0 -0.99963" />
@@ -369,5 +369,5 @@
   </joint>
   <link
-    name="lizi_$(arg lizi_id)/Right_URF_Link">
+    name="lizi_$(arg lizi_id)_Right_URF_link">
     <inertial>
       <origin
@@ -409,5 +409,5 @@
   </link>
   <joint
-    name="lizi_$(arg lizi_id)/Right_URF_Joint"
+    name="lizi_$(arg lizi_id)_Right_URF_Joint"
     type="fixed">
     <origin
@@ -415,12 +415,12 @@
       rpy="0 2.6072E-16 -1.57" />
     <parent
-      link="lizi_$(arg lizi_id)/base_link" />
-    <child
-      link="lizi_$(arg lizi_id)/Right_URF_Link" />
+      link="lizi_$(arg lizi_id)_base_link" />
+    <child
+      link="lizi_$(arg lizi_id)_Right_URF_link" />
     <axis
       xyz="0 0 0" />
   </joint>
   <link
-    name="lizi_$(arg lizi_id)/Left_URF_Link">
+    name="lizi_$(arg lizi_id)_Left_URF_link">
     <inertial>
       <origin
@@ -462,5 +462,5 @@
   </link>
   <joint
-    name="lizi_$(arg lizi_id)/Left_URF_Joint"
+    name="lizi_$(arg lizi_id)_Left_URF_Joint"
     type="fixed">
     <origin
@@ -468,12 +468,12 @@
       rpy="0 0 1.57" />
     <parent
-      link="lizi_$(arg lizi_id)/base_link" />
-    <child
-      link="lizi_$(arg lizi_id)/Left_URF_Link" />
+      link="lizi_$(arg lizi_id)_base_link" />
+    <child
+      link="lizi_$(arg lizi_id)_Left_URF_link" />
     <axis
       xyz="0 0 0" />
   </joint>
   <link
-    name="lizi_$(arg lizi_id)/Rear_URF_Link">
+    name="lizi_$(arg lizi_id)_Rear_URF_link">
     <inertial>
       <origin
@@ -515,5 +515,5 @@
   </link>
   <joint
-    name="lizi_$(arg lizi_id)/Rear_URF_Joint"
+    name="lizi_$(arg lizi_id)_Rear_URF_Joint"
     type="fixed">
     <origin
@@ -521,12 +521,12 @@
       rpy="0 0 3.14" />
     <parent
-      link="lizi_$(arg lizi_id)/base_link" />
-    <child
-      link="lizi_$(arg lizi_id)/Rear_URF_Link" />
+      link="lizi_$(arg lizi_id)_base_link" />
+    <child
+      link="lizi_$(arg lizi_id)_Rear_URF_link" />
     <axis
       xyz="0 0 0" />
   </joint>
   <link
-    name="lizi_$(arg lizi_id)/Laser_Link">
+    name="lizi_$(arg lizi_id)_Laser_link">
     <inertial>
       <origin
@@ -549,5 +549,5 @@
       <geometry>
         <mesh
-          filename="package://lizi/lizi_urdf/meshes/Laser_Link.STL" />
+          filename="package://lizi/lizi_urdf/meshes/Laser_link.STL" />
       </geometry>
       <material
@@ -563,10 +563,10 @@
       <geometry>
         <mesh
-          filename="package://lizi/lizi_urdf/meshes/Laser_Link.STL" />
-      </geometry>
-    </collision>
-  </link>
-  <joint
-    name="lizi_$(arg lizi_id)/Laser_Joint"
+          filename="package://lizi/lizi_urdf/meshes/Laser_link.STL" />
+      </geometry>
+    </collision>
+  </link>
+  <joint
+    name="lizi_$(arg lizi_id)_Laser_Joint"
     type="fixed">
     <origin
@@ -574,12 +574,12 @@
       rpy="2.1253E-16 8.5011E-16 -2.6741E-16" />
     <parent
-      link="lizi_$(arg lizi_id)/base_link" />
-    <child
-      link="lizi_$(arg lizi_id)/Laser_Link" />
+      link="lizi_$(arg lizi_id)_base_link" />
+    <child
+      link="lizi_$(arg lizi_id)_Laser_link" />
     <axis
       xyz="0 0 0" />
   </joint>
   <link
-    name="lizi_$(arg lizi_id)/Camera_Link">
+    name="lizi_$(arg lizi_id)_Camera_link">
     <inertial>
       <origin
@@ -621,5 +621,5 @@
   </link>
   <joint
-    name="lizi_$(arg lizi_id)/Camera_Joint"
+    name="lizi_$(arg lizi_id)_Camera_Joint"
     type="fixed">
     <origin
@@ -627,7 +627,7 @@
       rpy="1.6519E-18 -0.0061583 -2.6824E-16" />
     <parent
-      link="lizi_$(arg lizi_id)/base_link" />
-    <child
-      link="lizi_$(arg lizi_id)/Camera_Link" />
+      link="lizi_$(arg lizi_id)_base_link" />
+    <child
+      link="lizi_$(arg lizi_id)_Camera_link" />
     <axis
       xyz="0 0 0" />

Commit message: lizi color

File: lizi_urdf/robots/lizi.xacro (robot description, xacro)
@@ -1,4 +1,5 @@
 <?xml version="1.0"?>
 <robot xmlns:xacro="http://www.ros.org/wiki/lizi" name="lizi_urdf">
+<xacro:property name="lizi_color" value="0 0.517 0.26 1" />
   <link
     name="lizi_$(arg lizi_id)_base_link">
@@ -28,5 +29,5 @@
         name="">
         <color
-          rgba="0 0.517 0.26 1" />
+          rgba="${lizi_color}" />
       </material>
     </visual>

Commit message: order

File: lizi_urdf/robots/lizi.xacro (robot description, xacro)
@@ -1,5 +1,5 @@
 <?xml version="1.0"?>
-<robot xmlns:xacro="http://www.ros.org/wiki/lizi" name="lizi_urdf">
-<xacro:property name="lizi_color" value="0.72 0 0 1" />
+<robot xmlns:xacro="http://www.ros.org/wiki/lizi_robot" name="lizi_urdf">
+<xacro:property name="lizi_color" value="0 0.517 0.26 1" />
   <link
     name="lizi_$(arg lizi_id)_base_link">
@@ -24,5 +24,5 @@
       <geometry>
         <mesh
-          filename="package://lizi/lizi_urdf/meshes/base_link.STL" />
+          filename="package://lizi_urdf/meshes/base_link.STL" />
       </geometry>
       <material
@@ -38,5 +38,5 @@
       <geometry>
         <mesh
-          filename="package://lizi/lizi_urdf/meshes/base_link.STL" />
+          filename="package://lizi_urdf/meshes/base_link.STL" />
       </geometry>
     </collision>
@@ -64,5 +64,5 @@
       <geometry>
         <mesh
-          filename="package://lizi/lizi_urdf/meshes/FL_Wheel_Link.STL" />
+          filename="package://lizi_urdf/meshes/FL_Wheel_Link.STL" />
       </geometry>
       <material
@@ -78,5 +78,5 @@
       <geometry>
         <mesh
-          filename="package://lizi/lizi_urdf/meshes/FL_Wheel_Link.STL" />
+          filename="package://lizi_urdf/meshes/FL_Wheel_Link.STL" />
       </geometry>
     </collision>
@@ -117,5 +117,5 @@
       <geometry>
         <mesh
-          filename="package://lizi/lizi_urdf/meshes/RL_Wheel_Link.STL" />
+          filename="package://lizi_urdf/meshes/RL_Wheel_Link.STL" />
       </geometry>
       <material
@@ -131,5 +131,5 @@
       <geometry>
         <mesh
-          filename="package://lizi/lizi_urdf/meshes/RL_Wheel_Link.STL" />
+          filename="package://lizi_urdf/meshes/RL_Wheel_Link.STL" />
       </geometry>
     </collision>
@@ -173,5 +173,5 @@
       <geometry>
         <mesh
-          filename="package://lizi/lizi_urdf/meshes/RR_Wheel_Link.STL" />
+          filename="package://lizi_urdf/meshes/RR_Wheel_Link.STL" />
       </geometry>
       <material
@@ -187,5 +187,5 @@
       <geometry>
         <mesh
-          filename="package://lizi/lizi_urdf/meshes/RR_Wheel_Link.STL" />
+          filename="package://lizi_urdf/meshes/RR_Wheel_Link.STL" />
       </geometry>
     </collision>
@@ -226,5 +226,5 @@
       <geometry>
         <mesh
-          filename="package://lizi/lizi_urdf/meshes/FR_Wheel_Link.STL" />
+          filename="package://lizi_urdf/meshes/FR_Wheel_Link.STL" />
       </geometry>
       <material
@@ -240,5 +240,5 @@
       <geometry>
         <mesh
-          filename="package://lizi/lizi_urdf/meshes/FR_Wheel_Link.STL" />
+          filename="package://lizi_urdf/meshes/FR_Wheel_Link.STL" />
       </geometry>
     </collision>
@@ -279,5 +279,5 @@
       <geometry>
         <mesh
-          filename="package://lizi/lizi_urdf/meshes/Asus_Pan_Link.STL" />
+          filename="package://lizi_urdf/meshes/Asus_Pan_Link.STL" />
       </geometry>
       <material
@@ -293,5 +293,5 @@
       <geometry>
         <mesh
-          filename="package://lizi/lizi_urdf/meshes/Asus_Pan_Link.STL" />
+          filename="package://lizi_urdf/meshes/Asus_Pan_Link.STL" />
       </geometry>
     </collision>
@@ -335,5 +335,5 @@
       <geometry>
         <mesh
-          filename="package://lizi/lizi_urdf/meshes/Asus_Camera_Link.STL" />
+          filename="package://lizi_urdf/meshes/Asus_Camera_Link.STL" />
       </geometry>
       <material
@@ -349,5 +349,5 @@
       <geometry>
         <mesh
-          filename="package://lizi/lizi_urdf/meshes/Asus_Camera_Link.STL" />
+          filename="package://lizi_urdf/meshes/Asus_Camera_Link.STL" />
       </geometry>
     </collision>
@@ -391,5 +391,5 @@
       <geometry>
         <mesh
-          filename="package://lizi/lizi_urdf/meshes/Right_URF_Link.STL" />
+          filename="package://lizi_urdf/meshes/Right_URF_Link.STL" />
       </geometry>
       <material
@@ -405,5 +405,5 @@
       <geometry>
         <mesh
-          filename="package://lizi/lizi_urdf/meshes/Right_URF_Link.STL" />
+          filename="package://lizi_urdf/meshes/Right_URF_Link.STL" />
       </geometry>
     </collision>
@@ -444,5 +444,5 @@
       <geometry>
         <mesh
-          filename="package://lizi/lizi_urdf/meshes/Left_URF_Link.STL" />
+          filename="package://lizi_urdf/meshes/Left_URF_Link.STL" />
       </geometry>
       <material
@@ -458,5 +458,5 @@
       <geometry>
         <mesh
-          filename="package://lizi/lizi_urdf/meshes/Left_URF_Link.STL" />
+          filename="package://lizi_urdf/meshes/Left_URF_Link.STL" />
       </geometry>
     </collision>
@@ -497,5 +497,5 @@
       <geometry>
         <mesh
-          filename="package://lizi/lizi_urdf/meshes/Rear_URF_Link.STL" />
+          filename="package://lizi_urdf/meshes/Rear_URF_Link.STL" />
       </geometry>
       <material
@@ -511,5 +511,5 @@
       <geometry>
         <mesh
-          filename="package://lizi/lizi_urdf/meshes/Rear_URF_Link.STL" />
+          filename="package://lizi_urdf/meshes/Rear_URF_Link.STL" />
       </geometry>
     </collision>
@@ -550,5 +550,5 @@
       <geometry>
         <mesh
-          filename="package://lizi/lizi_urdf/meshes/Laser_Link.STL" />
+          filename="package://lizi_urdf/meshes/Laser_Link.STL" />
       </geometry>
       <material
@@ -564,5 +564,5 @@
       <geometry>
         <mesh
-          filename="package://lizi/lizi_urdf/meshes/Laser_Link.STL" />
+          filename="package://lizi_urdf/meshes/Laser_Link.STL" />
       </geometry>
     </collision>
@@ -603,5 +603,5 @@
       <geometry>
         <mesh
-          filename="package://lizi/lizi_urdf/meshes/Camera_Link.STL" />
+          filename="package://lizi_urdf/meshes/Camera_Link.STL" />
       </geometry>
       <material
@@ -617,5 +617,5 @@
       <geometry>
         <mesh
-          filename="package://lizi/lizi_urdf/meshes/Camera_Link.STL" />
+          filename="package://lizi_urdf/meshes/Camera_Link.STL" />
       </geometry>
     </collision>
